Commit message: 集成到其他的地图上

File: prius_integration/prius_scaled_description/urdf/prius_scaled.urdf (robot description, URDF)
Before this commit: robot prius_scaled, 12 links, 11 joints
Links:
- link front_left_wheel: geometry collision cylinder length=0.02 radius=0.031265; visual mesh filename=package://prius_scaled_description/meshes/wheel.obj scale=0.001 0.001 0.001
- link front_right_wheel: geometry collision cylinder length=0.02 radius=0.031265; visual mesh filename=package://prius_scaled_description/meshes/wheel.obj scale=0.001 0.001 0.001
- link rear_left_wheel: geometry collision cylinder length=0.02 radius=0.031265; visual mesh filename=package://prius_scaled_description/meshes/wheel.obj scale=0.001 0.001 0.001
- link rear_right_wheel: geometry collision cylinder length=0.02 radius=0.031265; visual mesh filename=package://prius_scaled_description/meshes/wheel.obj scale=0.001 0.001 0.001

Commit message: fix: prius模型集成到地图上显示，Rvix无报错

File: prius_integration/prius_scaled_description/urdf/prius_scaled.urdf (robot description, URDF)
Before this commit: robot prius_scaled, 12 links, 11 joints
Links:
- link front_left_wheel: geometry collision sphere radius=0.031265; visual mesh filename=package://prius_scaled_description/meshes/wheel.obj scale=0.001 0.001 0.001
- link front_right_wheel: geometry collision sphere radius=0.031265; visual mesh filename=package://prius_scaled_description/meshes/wheel.obj scale=0.001 0.001 0.001
- link rear_left_wheel: geometry collision sphere radius=0.031265; visual mesh filename=package://prius_scaled_description/meshes/wheel.obj scale=0.001 0.001 0.001
- link rear_right_wheel: geometry collision sphere radius=0.031265; visual mesh filename=package://prius_scaled_description/meshes/wheel.obj scale=0.001 0.001 0.001
Joints:
- joint front_left_steer_joint: type continuous -> revolute
- joint front_right_steer_joint: type continuous -> revolute
- joint steering_joint: limit lower=-7.85 upper=7.85 effort=10000000 velocity=1000000 -> lower=-6.28 upper=6.28 effort=10000000 velocity=1000000; type continuous -> revolute
